File: Controller.kicad_sch (KiCad schematic)
At the start: 43 parts, among them J1 Barrel_Jack_Switch, J2 USB-C, Q1 AO3401A, Q2 BC817, Q3 BC817, SW1 Power_SW, U1 ESP-32_Module, U2 LM2576S-5, U3 CH340G, U4 LM1117MP-3.3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

Commit message: Schematic Completed, Footprints Assigned
Parts:
- C1, C10, C11, C2, C3, C4, C5, C6, C8, C9: footprint (none) -> Capacitor_SMD:C_0805_2012Metric_Pad1.18x1.45mm_HandSolder
- D3, D4, D6: footprint (none) -> LED_SMD:LED_1206_3216Metric_ReverseMount_Hole1.8x2.4mm
- J1: footprint (none) -> Connector_BarrelJack:BarrelJack_Horizontal
- R1, R10, R11, R2, R3, R4, R5, R6, R7, R8: footprint (none) -> Resistor_SMD:R_0805_2012Metric_Pad1.20x1.40mm_HandSolder
- R9: footprint (none) -> Resistor_SMD:R_1206_3216Metric_Pad1.30x1.75mm_HandSolder
- Y1: footprint (none) -> Crystal:Crystal_HC49-4H_Vertical
Changed lines of the file:
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@@
 			)
 		)
-		(property "Footprint" ""
+		(property "Footprint" "Resistor_SMD:R_0805_2012Metric_Pad1.20x1.40mm_HandSolder"
 			(at 156.21 154.94 0)
 			(effects
@@
 			)
 		)
-		(property "Footprint" ""
+		(property "Footprint" "Capacitor_SMD:C_0805_2012Metric_Pad1.18x1.45mm_HandSolder"
 			(at 137.16 119.38 0)
 			(effects
@@
 			)
 		)
-		(property "Footprint" ""
+		(property "Footprint" "Capacitor_SMD:C_0805_2012Metric_Pad1.18x1.45mm_HandSolder"
 			(at 87.63 137.16 0)
 			(effects
@@
 			)
 		)
-		(property "Footprint" ""
+		(property "Footprint" "Connector_BarrelJack:BarrelJack_Horizontal"
 			(at 26.67 28.956 0)
 			(effects
@@
 			)
 		)
-		(property "Footprint" ""
+		(property "Footprint" "Resistor_SMD:R_0805_2012Metric_Pad1.20x1.40mm_HandSolder"
 			(at 210.82 95.25 0)
 			(effects
@@
 			)
 		)
-		(property "Footprint" ""
+		(property "Footprint" "Capacitor_SMD:C_0805_2012Metric_Pad1.18x1.45mm_HandSolder"
 			(at 91.44 36.83 0)
 			(effects
@@
 			)
 		)
-		(property "Footprint" ""
+		(property "Footprint" "LED_SMD:LED_1206_3216Metric_ReverseMount_Hole1.8x2.4mm"
 			(at 156.21 163.83 90)
 			(effects
@@
 			)
 		)
-		(property "Footprint" ""
+		(property "Footprint" "Resistor_SMD:R_0805_2012Metric_Pad1.20x1.40mm_HandSolder"
 			(at 271.78 46.99 0)
 			(effects
@@
 			)
 		)
-		(property "Footprint" ""
+		(property "Footprint" "Resistor_SMD:R_0805_2012Metric_Pad1.20x1.40mm_HandSolder"
 			(at 245.11 53.34 0)
 			(effects
@@
 			)
 		)
-		(property "Footprint" ""
+		(property "Footprint" "Resistor_SMD:R_1206_3216Metric_Pad1.30x1.75mm_HandSolder"
 			(at 229.87 121.92 0)
 			(effects
@@
 			)
 		)
-		(property "Footprint" ""
+		(property "Footprint" "Capacitor_SMD:C_0805_2012Metric_Pad1.18x1.45mm_HandSolder"
 			(at 88.9 97.79 0)
 			(effects
@@
 			)
 		)
-		(property "Footprint" ""
+		(property "Footprint" "Resistor_SMD:R_0805_2012Metric_Pad1.20x1.40mm_HandSolder"
 			(at 138.43 154.94 0)
 			(effects
@@
 			)
 		)
-		(property "Footprint" ""
+		(property "Footprint" "Capacitor_SMD:C_0805_2012Metric_Pad1.18x1.45mm_HandSolder"
 			(at 76.2 97.79 0)
 			(effects
@@
 			)
 		)
-		(property "Footprint" ""
+		(property "Footprint" "Resistor_SMD:R_0805_2012Metric_Pad1.20x1.40mm_HandSolder"
 			(at 95.25 124.46 0)
 			(effects
@@
 			)
 		)
-		(property "Footprint" ""
+		(property "Footprint" "Capacitor_SMD:C_0805_2012Metric_Pad1.18x1.45mm_HandSolder"
 			(at 199.39 45.72 0)
 			(effects
@@
 			)
 		)
-		(property "Footprint" ""
+		(property "Footprint" "Resistor_SMD:R_0805_2012Metric_Pad1.20x1.40mm_HandSolder"
 			(at 130.81 184.15 0)
 			(effects
@@
 			)
 		)
-		(property "Footprint" ""
+		(property "Footprint" "LED_SMD:LED_1206_3216Metric_ReverseMount_Hole1.8x2.4mm"
 			(at 245.11 45.72 90)
 			(effects
@@
 			)
 		)
-		(property "Footprint" ""
+		(property "Footprint" "Resistor_SMD:R_0805_2012Metric_Pad1.20x1.40mm_HandSolder"
 			(at 166.37 45.72 0)
 			(effects
@@
 			)
 		)
-		(property "Footprint" ""
+		(property "Footprint" "Resistor_SMD:R_0805_2012Metric_Pad1.20x1.40mm_HandSolder"
 			(at 133.35 172.72 0)
 			(effects
@@
 			)
 		)
-		(property "Footprint" ""
+		(property "Footprint" "Crystal:Crystal_HC49-4H_Vertical"
 			(at 148.59 124.46 0)
 			(effects
@@
 			)
 		)
-		(property "Footprint" ""
+		(property "Footprint" "Capacitor_SMD:C_0805_2012Metric_Pad1.18x1.45mm_HandSolder"
 			(at 137.16 132.08 0)
 			(effects
@@
 			)
 		)
-		(property "Footprint" ""
+		(property "Footprint" "LED_SMD:LED_1206_3216Metric_ReverseMount_Hole1.8x2.4mm"
 			(at 138.43 163.83 90)
 			(effects
@@
 			)
 		)
-		(property "Footprint" ""
+		(property "Footprint" "Resistor_SMD:R_0805_2012Metric_Pad1.20x1.40mm_HandSolder"
 			(at 210.82 128.27 0)
 			(effects
@@
 			)
 		)
-		(property "Footprint" ""
+		(property "Footprint" "Capacitor_SMD:C_0805_2012Metric_Pad1.18x1.45mm_HandSolder"
 			(at 228.6 44.45 0)
 			(effects
@@
 			)
 		)
-		(property "Footprint" ""
+		(property "Footprint" "Capacitor_SMD:C_0805_2012Metric_Pad1.18x1.45mm_HandSolder"
 			(at 176.53 93.98 0)
 			(effects
@@
 			)
 		)
-		(property "Footprint" ""
+		(property "Footprint" "Capacitor_SMD:C_0805_2012Metric_Pad1.18x1.45mm_HandSolder"
 			(at 237.49 44.45 0)
 			(effects

Commit message: Symbol and footprint library exported
Parts:
- C1, C10, C11, C2, C3, C5, C6, C8, C9: symbol Device:C_Small -> ESP32_Xbee_LoRa:C_Small
- C4: symbol Device:C_Polarized_Small -> ESP32_Xbee_LoRa:C_Polarized_Small
- C7: symbol LOGSUN:LGS-KC-SMD&DIP -> ESP32_Xbee_LoRa:LGS-KC-SMD&DIP
- D1: symbol Diode_Bridge:W10G -> ESP32_Xbee_LoRa:W10G
- D2: symbol Diode:1N5822 -> ESP32_Xbee_LoRa:1N5822
- D3, D4, D6: symbol Device:LED_Small -> ESP32_Xbee_LoRa:LED_Small
- D5: symbol Diode:1N5819 -> ESP32_Xbee_LoRa:1N5819
- D7, D8: symbol Diode:BAT54C -> ESP32_Xbee_LoRa:BAT54C
- J1: symbol Connector:Barrel_Jack_Switch -> ESP32_Xbee_LoRa:Barrel_Jack_Switch
- J2: symbol LOGSUN:LGS-KC-CSP-USC16-TR -> ESP32_Xbee_LoRa:LGS-KC-CSP-USC16-TR
- L1: symbol LOGSUN:LGS-KC-DIL4 -> ESP32_Xbee_LoRa:LGS-KC-DIL4
- Q1: symbol Transistor_FET:AO3401A -> ESP32_Xbee_LoRa:AO3401A
- Q2, Q3: symbol Transistor_BJT:BC817 -> ESP32_Xbee_LoRa:BC817
- R1, R10, R11, R2, R3, R4, R5, R6, R7, R8, R9: symbol Device:R_Small -> ESP32_Xbee_LoRa:R_Small
- S1: symbol LOGSUN:LGS-KC-10-XX -> ESP32_Xbee_LoRa:LGS-KC-10-XX
- SW1: symbol LOGSUN:LGS-KC-SW -> ESP32_Xbee_LoRa:LGS-KC-SW
- U1: symbol NITIN:esp32_wroom_module -> ESP32_Xbee_LoRa:esp32_wroom_module
- U2: symbol Regulator_Switching:LM2576S-5 -> ESP32_Xbee_LoRa:LM2576S-5
- U3: symbol Interface_USB:CH340G -> ESP32_Xbee_LoRa:CH340G
- U4: symbol Regulator_Linear:LM1117MP-3.3 -> ESP32_Xbee_LoRa:LM1117MP-3.3
- Y1: symbol Device:Crystal_Small -> ESP32_Xbee_LoRa:Crystal_Small
