File: ESP32_Xbee_Lora.kicad_pcb (KiCad board)
At the start: 2 copper layers, 200 x 160 mm, 129 parts, among them J1 Barrel_Jack_Switch, J10 RGB, J11 Conn_01x03_Pin, J12 Conn_01x03_Pin, J13 I2C, J14 UART, J15 RGB, J16 POT, J2 USB-C, J3 Relay_1, J4 Relay_2, J5 RELAY, J6 OLED, J7 LM_35, J8 LDR, J9 POT, K1 SANYOU_SRD_Form_C, K2 SANYOU_SRD_Form_C, M1 Wireless_Module, Q1 AO3401A, Q2 BC817, Q3 BC817, Q4 BC847, Q5 BC847, Q6 BC858, Q7 BC858, SW1 Power_SW, U1 ESP-32_Module, U2 LM2576S-5, U3 CH340G, U4 LM1117MP-3.3, U5 0.96" OLED(I2C), U6 LM35-LP, U7 LM1117MP-3.3, Y1 12MHz

Commit message: Tentative Placement Done
Parts:
- added H1: MountingHole, MountingHole:MountingHole_3.2mm_M3_Pad_Via, F.Cu at (105.4, 66.0)
- added H2: MountingHole, MountingHole:MountingHole_3.2mm_M3_Pad_Via, F.Cu at (106.3, 215.5)
- added H3: MountingHole, MountingHole:MountingHole_3.2mm_M3_Pad_Via, F.Cu at (296.3, 64.3)
- added H4: MountingHole, MountingHole:MountingHole_3.2mm_M3_Pad_Via, F.Cu at (295.8, 217.2)
- added R41: 1K, Resistor_SMD:R_0805_2012Metric_Pad1.20x1.40mm_HandSolder, F.Cu at (190.2, 120.2)
- added R42: 1K, Resistor_SMD:R_0805_2012Metric_Pad1.20x1.40mm_HandSolder, F.Cu at (190.2, 123.2)
- added R43: 1K, Resistor_SMD:R_0805_2012Metric_Pad1.20x1.40mm_HandSolder, F.Cu at (190.2, 126.1)
- added R44: 1K, Resistor_SMD:R_0805_2012Metric_Pad1.20x1.40mm_HandSolder, F.Cu at (190.2, 129.1)
- added R45: 1K, Resistor_SMD:R_0805_2012Metric_Pad1.20x1.40mm_HandSolder, F.Cu at (190.2, 132.0)
- added R46: 1K, Resistor_SMD:R_0805_2012Metric_Pad1.20x1.40mm_HandSolder, F.Cu at (190.2, 135.0)
- added R47: 1K, Resistor_SMD:R_0805_2012Metric_Pad1.20x1.40mm_HandSolder, F.Cu at (195.0, 120.2)
- added R48: 1K, Resistor_SMD:R_0805_2012Metric_Pad1.20x1.40mm_HandSolder, F.Cu at (195.0, 123.2)
- added R49: 1K, Resistor_SMD:R_0805_2012Metric_Pad1.20x1.40mm_HandSolder, F.Cu at (195.0, 126.1)
- added R50: 1K, Resistor_SMD:R_0805_2012Metric_Pad1.20x1.40mm_HandSolder, F.Cu at (195.0, 129.1)
- C12, C13, C14, U4, U7: moved to B.Cu
- D10, D11, D12, D13, D14, D15, D16, D9: footprint LED_SMD:LED_1206_3216Metric_ReverseMount_Hole1.8x2.4mm -> LED_SMD:LED_1206_3216Metric_Pad1.42x1.75mm_HandSolder
- moved R40 508.0 mm to (310.4, 462.0), turned to 90 degrees
- moved Q4 405.0 mm to (249.8, 129.9)
- moved Q5 405.0 mm to (249.8, 134.3)
- moved Q6 405.0 mm to (249.8, 138.8)
- moved Q7 405.0 mm to (249.8, 143.2)
- moved D18 397.0 mm to (265.4, 139.7), turned to 90 degrees
- moved D17 393.4 mm to (261.9, 139.7), turned to 90 degrees
- moved R28 392.3 mm to (256.8, 125.4)
- moved R29 392.3 mm to (256.8, 128.3)
- moved R30 392.3 mm to (256.8, 131.3)
- moved R31 392.3 mm to (256.8, 134.2)
- moved R32 392.3 mm to (256.8, 137.2)
- moved R33 392.3 mm to (256.8, 140.2)
- moved R34 392.3 mm to (256.8, 143.1)
- moved R35 392.3 mm to (256.8, 146.1)
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Connections:
- BAR1 pad 1: /OLED_Relays/BAR 1 -> /OLED_Relays/BAR 10
- BAR1 pad 10: /OLED_Relays/BAR 10 -> /OLED_Relays/BAR 1
- BAR1 pad 2: /OLED_Relays/BAR 2 -> /OLED_Relays/BAR 9
- BAR1 pad 3: /OLED_Relays/BAR 3 -> /OLED_Relays/BAR 8
- BAR1 pad 4: /OLED_Relays/BAR 4 -> /OLED_Relays/BAR 7
- BAR1 pad 5: /OLED_Relays/BAR 5 -> /OLED_Relays/BAR 6
- BAR1 pad 6: /OLED_Relays/BAR 6 -> /OLED_Relays/BAR 5
- BAR1 pad 7: /OLED_Relays/BAR 7 -> /OLED_Relays/BAR 4
- BAR1 pad 8: /OLED_Relays/BAR 8 -> /OLED_Relays/BAR 3
- BAR1 pad 9: /OLED_Relays/BAR 9 -> /OLED_Relays/BAR 2
- SV2 pad 3: unconnected-(SV2-Pad3) -> /OLED_Relays/LD 9
- SV2 pad 4: unconnected-(SV2-Pad4) -> /OLED_Relays/LD 10

Commit message: Symbol and footprint library exported
Parts:
- BAR1: footprint Display:HDSP-4830 -> ESP32_Xbee_LoRa:HDSP-4830
- C1, C10, C11, C12, C13, C14, C2, C3, C4, C5, C6, C8, C9: footprint Capacitor_SMD:C_0805_2012Metric_Pad1.18x1.45mm_HandSolder -> ESP32_Xbee_LoRa:C_0805_2012Metric_Pad1.18x1.45mm_HandSolder
- C7: footprint LOGSUN:LGS-KC-140CLH-1010 -> ESP32_Xbee_LoRa:LGS-KC-140CLH-1010
- D1: footprint Diode_THT:Diode_Bridge_Round_D9.8mm -> ESP32_Xbee_LoRa:Diode_Bridge_Round_D9.8mm
- D10, D11, D12, D13, D14, D15, D16, D9: footprint LED_SMD:LED_1206_3216Metric_Pad1.42x1.75mm_HandSolder -> ESP32_Xbee_LoRa:LED_1206_3216Metric_Pad1.42x1.75mm_HandSolder
- D17, D18: footprint Diode_THT:D_DO-35_SOD27_P7.62mm_Horizontal -> ESP32_Xbee_LoRa:D_DO-35_SOD27_P7.62mm_Horizontal
- D19: footprint LOGSUN:LGS-KC-LED5MMRGB -> ESP32_Xbee_LoRa:LGS-KC-LED5MMRGB
- D2: footprint Diode_THT:D_DO-201AD_P15.24mm_Horizontal -> ESP32_Xbee_LoRa:D_DO-201AD_P15.24mm_Horizontal
- D3, D4, D6: footprint LED_SMD:LED_1206_3216Metric_ReverseMount_Hole1.8x2.4mm -> ESP32_Xbee_LoRa:LED_1206_3216Metric_ReverseMount_Hole1.8x2.4mm
- D5: footprint Diode_THT:D_DO-41_SOD81_P10.16mm_Horizontal -> ESP32_Xbee_LoRa:D_DO-41_SOD81_P10.16mm_Horizontal
- D7, D8, Q1, Q2, Q3, Q4, Q5, Q6, Q7: footprint Package_TO_SOT_SMD:SOT-23 -> ESP32_Xbee_LoRa:SOT-23
- H1, H2, H3, H4: footprint MountingHole:MountingHole_3.2mm_M3_Pad_Via -> ESP32_Xbee_LoRa:MountingHole_3.2mm_M3_Pad_Via
- J1: footprint Connector_BarrelJack:BarrelJack_Horizontal -> ESP32_Xbee_LoRa:BarrelJack_Horizontal
- J10, J15, J16, J9: footprint Connector_JST:JST_EH_B5B-EH-A_1x05_P2.50mm_Vertical -> ESP32_Xbee_LoRa:JST_EH_B5B-EH-A_1x05_P2.50mm_Vertical
- J11, J12, J7, J8: footprint Connector_JST:JST_EH_B3B-EH-A_1x03_P2.50mm_Vertical -> ESP32_Xbee_LoRa:JST_EH_B3B-EH-A_1x03_P2.50mm_Vertical
- J13, J14, J5, J6: footprint Connector_JST:JST_EH_B4B-EH-A_1x04_P2.50mm_Vertical -> ESP32_Xbee_LoRa:JST_EH_B4B-EH-A_1x04_P2.50mm_Vertical
- J2: footprint LOGSUN:LGS-KC-VALCON_CSP-USC16-TR -> ESP32_Xbee_LoRa:LGS-KC-VALCON_CSP-USC16-TR
- J3, J4: footprint TerminalBlock_Phoenix:TerminalBlock_Phoenix_MKDS-1,5-3-5.08_1x03_P5.08mm_Horizontal -> ESP32_Xbee_LoRa:TerminalBlock_Phoenix_MKDS-1,5-3-5.08_1x03_P5.08mm_Horizontal
- K1, K2: footprint LOGSUN:LGS-KC-FRS1B -> ESP32_Xbee_LoRa:LGS-KC-FRS1B
- L1: footprint LOGSUN:LGS-KC-MS42 -> ESP32_Xbee_LoRa:LGS-KC-MS42
- M1: footprint LOGSUN:LGS-KC-Wireless_Mod -> ESP32_Xbee_LoRa:LGS-KC-Wireless_Mod
- R1, R10, R11, R12, R13, R14, R15, R16, R17, R18, R19, R2, R20, R21, R22, R23, R24, R25, R26, R27, R28, R29, R3, R30, R31, R32, R33, R34, R35, R36, R37, R38, R4, R40, R41, R42, R43, R44, R45, R46, R47, R48, R49, R5, R50, R6, R7, R8: footprint Resistor_SMD:R_0805_2012Metric_Pad1.20x1.40mm_HandSolder -> ESP32_Xbee_LoRa:R_0805_2012Metric_Pad1.20x1.40mm_HandSolder
- R39: footprint OptoDevice:R_LDR_5.1x4.3mm_P3.4mm_Vertical -> ESP32_Xbee_LoRa:R_LDR_5.1x4.3mm_P3.4mm_Vertical
- R9: footprint Resistor_SMD:R_1206_3216Metric_Pad1.30x1.75mm_HandSolder -> ESP32_Xbee_LoRa:R_1206_3216Metric_Pad1.30x1.75mm_HandSolder
- RV1, RV2, RV3: footprint LOGSUN:LGS-KC-CA6V -> ESP32_Xbee_LoRa:LGS-KC-CA6V
- S1, S2, S3, S4, S5, S6, S7, S8, S9: footprint LOGSUN:LGS-KC-B3F-10XX -> ESP32_Xbee_LoRa:LGS-KC-B3F-10XX
- SV1, SV2, SV3, SV4: footprint LOGSUN:LGS-KC-ML10_INTERFACE -> ESP32_Xbee_LoRa:LGS-KC-ML10_INTERFACE
- SV5, SV6, SV7: footprint LOGSUN:LGS-KC-ML10-CONTROLLER -> ESP32_Xbee_LoRa:LGS-KC-ML10-CONTROLLER
- SW1: footprint LOGSUN:LGS-KC-SLIDE -> ESP32_Xbee_LoRa:LGS-KC-SLIDE
- U1: footprint nitin:esp 32 wroom module -> ESP32_Xbee_LoRa:esp 32 wroom module
- U2: footprint Package_TO_SOT_SMD:TO-263-5_TabPin3 -> ESP32_Xbee_LoRa:TO-263-5_TabPin3
- U3: footprint Package_SO:SOIC-16_3.9x9.9mm_P1.27mm -> ESP32_Xbee_LoRa:SOIC-16_3.9x9.9mm_P1.27mm
- U4, U7: footprint Package_TO_SOT_SMD:SOT-223-3_TabPin2 -> ESP32_Xbee_LoRa:SOT-223-3_TabPin2
- U5: footprint nitin:OLED I2C -> ESP32_Xbee_LoRa:OLED I2C
- U6: footprint Package_TO_SOT_THT:TO-92_Inline -> ESP32_Xbee_LoRa:TO-92_Inline
- Y1: footprint Crystal:Crystal_HC49-4H_Vertical -> ESP32_Xbee_LoRa:Crystal_HC49-4H_Vertical
